File: pcb/Oszillatoren.kicad_pcb (KiCad board)
At the start: 2 copper layers, 100 x 55 mm, 67 parts, among them J1 Conn_01x01_Pin, J10 Conn_01x01_Pin, J11 Conn_01x01_Pin, J12 Conn_01x01_Pin, J13 Conn_01x01_Pin, J14 Conn_01x01_Pin, J15 Conn_01x01_Pin, J16 Conn_01x01_Pin, J17 Conn_01x01_Pin, J18 Conn_01x01_Pin, J19 Conn_01x01_Pin, J2 Conn_01x01_Pin, J3 Conn_01x01_Pin, J4 Conn_01x01_Pin, J5 Conn_01x01_Pin, J6 Conn_01x01_Pin, J7 Conn_01x01_Pin, J8 Conn_01x01_Pin, J9 Conn_01x01_Pin, U1 74AHC1G4210, U2 40106, U3 LM358, U4 LM358, Y1 Crystal, Y2 Crystal

Commit message: Changable Rs fixed
Parts:
- R12, R13, R2, R3, R5, R7, R8, R9: value changeable -> 10k

Commit message: all changable Rs fixed
Parts:
- R14, R4, R6: value changeable -> 10k
Changed lines of the file:
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@@
 			)
 		)
-		(property "Value" "changeable"
+		(property "Value" "10k"
 			(at 4.03 4.91 0)
 			(unlocked yes)
@@
 			)
 		)
-		(property "Description" "Resistor"
+		(property "Description" "changeable"
 			(at 0 0 0)
 			(layer "F.Fab")
@@
 			)
 		)
-		(property "Value" "changeable"
+		(property "Value" "10k"
 			(at 4.03 4.91 0)
 			(unlocked yes)
@@
 			)
 		)
-		(property "Description" "Resistor"
+		(property "Description" "changeable"
 			(at 0 0 0)
 			(layer "F.Fab")
@@
 			)
 		)
-		(property "Value" "changeable"
+		(property "Value" "10k"
 			(at 4.03 4.91 270)
 			(unlocked yes)
@@
 			)
 		)
-		(property "Description" "Resistor"
+		(property "Description" "changeable"
 			(at 0 0 90)
 			(layer "F.Fab")
