File: pcb/Oszillatoren.kicad_pcb (KiCad board)
At the start: 2 copper layers, 100 x 55 mm, 67 parts, among them J1 Conn_01x01_Pin, J10 Conn_01x01_Pin, J11 Conn_01x01_Pin, J12 Conn_01x01_Pin, J13 Conn_01x01_Pin, J14 Conn_01x01_Pin, J15 Conn_01x01_Pin, J16 Conn_01x01_Pin, J17 Conn_01x01_Pin, J18 Conn_01x01_Pin, J19 Conn_01x01_Pin, J2 Conn_01x01_Pin, J3 Conn_01x01_Pin, J4 Conn_01x01_Pin, J5 Conn_01x01_Pin, J6 Conn_01x01_Pin, J7 Conn_01x01_Pin, J8 Conn_01x01_Pin, J9 Conn_01x01_Pin, U1 74AHC1G4210, U2 40106, U3 LM358, U4 LM358, Y1 Crystal, Y2 Crystal

Commit message: Changable R: 3D-Model added
Parts:
- R15: value changeable -> 10k
