File: pcb/Oszillatoren.kicad_sch (KiCad schematic)
At the start: 67 parts, among them J1 Conn_01x01_Pin, J10 Conn_01x01_Pin, J11 Conn_01x01_Pin, J12 Conn_01x01_Pin, J13 Conn_01x01_Pin, J14 Conn_01x01_Pin, J15 Conn_01x01_Pin, J16 Conn_01x01_Pin, J17 Conn_01x01_Pin, J18 Conn_01x01_Pin, J19 Conn_01x01_Pin, J2 Conn_01x01_Pin, J3 Conn_01x01_Pin, J4 Conn_01x01_Pin, J5 Conn_01x01_Pin, J6 Conn_01x01_Pin, J7 Conn_01x01_Pin, J8 Conn_01x01_Pin, J9 Conn_01x01_Pin, U1 74AHC1G4210, U2 40106, U3 LM358, U4 LM358, Y1 Crystal, Y2 Crystal

Commit message: Changable Rs fixed
Parts:
- R12, R13, R2, R3, R5, R7, R8, R9: value changeable -> 10k
Changed lines of the file:
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@@
 			)
 		)
-		(property "Value" "changeable"
+		(property "Value" "10k"
 			(at 147.32 33.02 90)
+			(hide yes)
 			(show_name no)
 			(do_not_autoplace no)
@@
 			)
 		)
-		(property "Description" "Resistor"
-			(at 142.24 35.56 0)
-			(hide yes)
+		(property "Description" "changeable"
+			(at 141.986 32.766 90)
 			(show_name no)
 			(do_not_autoplace no)
@@
 			)
 		)
-		(property "Value" "changeable"
+		(property "Value" "10k"
 			(at 208.28 59.69 90)
+			(hide yes)
 			(show_name no)
 			(do_not_autoplace no)
@@
 			)
 		)
-		(property "Description" "Resistor"
-			(at 203.2 62.23 0)
-			(hide yes)
+		(property "Description" "changeable"
+			(at 203.2 64.77 90)
 			(show_name no)
 			(do_not_autoplace no)
@@
 			)
 		)
-		(property "Value" "changeable"
+		(property "Value" "10k"
 			(at 111.76 53.34 90)
+			(hide yes)
 			(show_name no)
 			(do_not_autoplace no)
@@
 			)
 		)
-		(property "Description" "Resistor"
-			(at 114.3 58.42 0)
-			(hide yes)
+		(property "Description" "changeable"
+			(at 110.998 59.182 90)
 			(show_name no)
 			(do_not_autoplace no)
@@
 			)
 		)
-		(property "Value" "changeable"
+		(property "Value" "10k"
 			(at 207.01 35.56 90)
+			(hide yes)
 			(show_name no)
 			(do_not_autoplace no)
@@
 			)
 		)
-		(property "Description" "Resistor"
-			(at 201.93 38.1 0)
-			(hide yes)
+		(property "Description" "changeable"
+			(at 202.692 35.306 90)
 			(show_name no)
 			(do_not_autoplace no)
@@
 			)
 		)
-		(property "Value" "changeable"
+		(property "Value" "10k"
 			(at 76.2 63.5 90)
+			(hide yes)
 			(show_name no)
 			(do_not_autoplace no)
@@
 			)
 		)
-		(property "Description" "Resistor"
-			(at 73.66 58.42 0)
-			(hide yes)
+		(property "Description" "changeable"
+			(at 76.708 59.182 90)
 			(show_name no)
 			(do_not_autoplace no)
@@
 			)
 		)
-		(property "Value" "changeable"
+		(property "Value" "10k"
 			(at 90.17 63.5 90)
+			(hide yes)
 			(show_name no)
 			(do_not_autoplace no)
@@
 			)
 		)
-		(property "Description" "Resistor"
-			(at 87.63 58.42 0)
-			(hide yes)
+		(property "Description" "changeable"
+			(at 90.932 58.674 90)
 			(show_name no)
 			(do_not_autoplace no)
@@
 			)
 		)
-		(property "Value" "changeable"
+		(property "Value" "10k"
 			(at 148.59 57.15 90)
+			(hide yes)
 			(show_name no)
 			(do_not_autoplace no)
@@
 			)
 		)
-		(property "Description" "Resistor"
-			(at 143.51 59.69 0)
-			(hide yes)
+		(property "Description" "changeable"
+			(at 143.51 62.23 90)
 			(show_name no)
 			(do_not_autoplace no)
@@
 			)
 		)
-		(property "Value" "changeable"
+		(property "Value" "10k"
 			(at 62.23 63.5 90)
+			(hide yes)
 			(show_name no)
 			(do_not_autoplace no)
@@
 			)
 		)
-		(property "Description" "Resistor"
-			(at 59.69 58.42 0)
-			(hide yes)
+		(property "Description" "changeable"
+			(at 62.738 58.674 90)
 			(show_name no)
 			(do_not_autoplace no)

Commit message: all changable Rs fixed
Parts:
- R14, R4, R6: value changeable -> 10k
Changed lines of the file:
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@@
 			)
 		)
-		(property "Value" "changeable"
+		(property "Value" "10k"
 			(at 43.18 33.02 90)
+			(hide yes)
 			(show_name no)
 			(do_not_autoplace no)
@@
 			)
 		)
-		(property "Description" "Resistor"
-			(at 38.1 35.56 0)
-			(hide yes)
+		(property "Description" "changeable"
+			(at 38.354 32.766 90)
 			(show_name no)
 			(do_not_autoplace no)
@@
 			)
 		)
-		(property "Value" "changeable"
+		(property "Value" "10k"
 			(at 48.26 99.06 90)
+			(hide yes)
 			(show_name no)
 			(do_not_autoplace no)
@@
 			)
 		)
-		(property "Description" "Resistor"
-			(at 43.18 101.6 0)
-			(hide yes)
+		(property "Description" "changeable"
+			(at 43.18 98.552 90)
 			(show_name no)
 			(do_not_autoplace no)
@@
 			)
 		)
-		(property "Value" "changeable"
+		(property "Value" "10k"
 			(at 43.18 39.37 90)
+			(hide yes)
 			(show_name no)
 			(do_not_autoplace no)
@@
 			)
 		)
-		(property "Description" "Resistor"
-			(at 38.1 41.91 0)
-			(hide yes)
+		(property "Description" "changeable"
+			(at 38.862 39.37 90)
 			(show_name no)
 			(do_not_autoplace no)

Commit message: Changable R: 3D-Model added
Parts:
- R15: value changeable -> 10k
Changed lines of the file:
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@@
 			)
 		)
-		(property "Value" "changeable"
+		(property "Value" "10k"
 			(at 21.59 114.3 90)
+			(hide yes)
 			(show_name no)
 			(do_not_autoplace no)
@@
 			)
 		)
-		(property "Description" "Resistor"
-			(at 24.13 119.38 0)
-			(hide yes)
+		(property "Description" "changeable"
+			(at 20.828 119.38 90)
 			(show_name no)
 			(do_not_autoplace no)
